File: 2tonewatch.kicad_pcb (KiCad board)
At the start: 2 copper layers, 0 parts

Commit message: Added layout rules and constraints
Parts:
- added AE1: 2450AT18A0100001E, LibraryFootprints:XCVR_2450AT18A0100001E, F.Cu at (128.2, 101.0)
- added C1: 4u7, Capacitor_SMD:C_0603_1608Metric, F.Cu at (135.4, 86.2)
- added C10: 4u7, Capacitor_SMD:C_0603_1608Metric, F.Cu at (135.4, 88.7)
- added C11: 100nF, Capacitor_SMD:C_0402_1005Metric, F.Cu at (131.9, 86.0)
- added C12: 100nF, Capacitor_SMD:C_0402_1005Metric, F.Cu at (131.9, 87.9)
- added C13: 4u7, Capacitor_SMD:C_0603_1608Metric, F.Cu at (135.4, 91.2)
- added C14: 10pF, Capacitor_SMD:C_0402_1005Metric, F.Cu at (131.9, 89.9)
- added C15: 10pF, Capacitor_SMD:C_0402_1005Metric, F.Cu at (131.9, 91.9)
- added C16: 1uF, Capacitor_SMD:C_0402_1005Metric, F.Cu at (154.4, 62.0)
- added C17: 0.1uF, Capacitor_SMD:C_0402_1005Metric, F.Cu at (154.4, 63.9)
- added C18: 1uF, Capacitor_SMD:C_0402_1005Metric, F.Cu at (154.4, 65.9)
- added C19: 1uF, Capacitor_SMD:C_0402_1005Metric, F.Cu at (154.4, 67.9)
- added C2: 100nF, Capacitor_SMD:C_0402_1005Metric, F.Cu at (126.2, 86.0)
- added C20: 1uF, Capacitor_SMD:C_0603_1608Metric, F.Cu at (117.1, 70.0)
- added C21: 4u7, Capacitor_SMD:C_0603_1608Metric, F.Cu at (117.1, 72.5)
- added C22: 4u7, Capacitor_SMD:C_0603_1608Metric, F.Cu at (117.1, 75.0)
- added C23: 1uF, Capacitor_SMD:C_0603_1608Metric, F.Cu at (117.1, 77.5)
- added C24: 1uF, Capacitor_SMD:C_0603_1608Metric, F.Cu at (121.1, 70.0)
- added C25: 1uF, Capacitor_SMD:C_0603_1608Metric, F.Cu at (121.1, 72.5)
- added C26: 1uF, Capacitor_SMD:C_0603_1608Metric, F.Cu at (121.1, 75.0)
- added C27: 1uF, Capacitor_SMD:C_0603_1608Metric, F.Cu at (121.1, 77.5)
- added C28: 1uF, Capacitor_SMD:C_0603_1608Metric, F.Cu at (125.1, 70.0)
- added C29: 1uF, Capacitor_SMD:C_0603_1608Metric, F.Cu at (125.1, 72.5)
- added C3: 100nF, Capacitor_SMD:C_0402_1005Metric, F.Cu at (126.2, 87.9)
- added C4: 100nF, Capacitor_SMD:C_0402_1005Metric, F.Cu at (126.2, 89.9)
- added C5: 100nF, Capacitor_SMD:C_0402_1005Metric, F.Cu at (126.2, 91.9)
- added C6: 100nF, Capacitor_SMD:C_0402_1005Metric, F.Cu at (129.1, 86.0)
- added C7: 100nF, Capacitor_SMD:C_0402_1005Metric, F.Cu at (129.1, 87.9)
- added C8: 100nF, Capacitor_SMD:C_0402_1005Metric, F.Cu at (129.1, 89.9)
- added C9: 100nF, Capacitor_SMD:C_0402_1005Metric, F.Cu at (129.1, 91.9)
- added D1: MBR0530, Diode_SMD:D_SOD-123, F.Cu at (130.0, 70.4)
- added D2: MBR0530, Diode_SMD:D_SOD-123, F.Cu at (130.0, 73.8)
- added D3: MBR0530, Diode_SMD:D_SOD-123, F.Cu at (130.0, 77.1)
- added J1: Conn_ARM_SWD_TagConnect_TC2030, Connector:Tag-Connect_TC2030-IDC-FP_2x03_P1.27mm_Vertical, F.Cu at (119.8, 99.1)
- added J2: USB_C_Receptacle_USB2.0_16P, Connector_USB:USB_C_Receptacle_Molex_105450-0101, F.Cu at (147.2, 66.0)
- added J3: Conn_01x02_Pin, Connector_JST:JST_PH_B2B-PH-K_1x02_P2.00mm_Vertical, F.Cu at (144.3, 74.2)
- added J4: FFC-FPC_1X24_PIN, Connector_FFC-FPC:Amphenol_F32Q-1A7x1-11024_1x24-1MP_P0.5mm_Horizontal, F.Cu at (125.7, 65.5)
- added L1: 10nH, Inductor_SMD:L_0402_1005Metric, F.Cu at (135.6, 100.4)
- added L2: 10uH, Inductor_SMD:L_0805_2012Metric, F.Cu at (135.1, 97.5)
- added L3: 47uH 500mA, Inductor_SMD:L_1210_3225Metric, F.Cu at (117.9, 80.9)
- added Q1: Si1308EDL, Package_TO_SOT_SMD:SOT-323_SC-70, F.Cu at (123.0, 80.7)
- added R10: 2R2, Resistor_SMD:R_0603_1608Metric, F.Cu at (125.1, 77.5)
- added R11: 1K, Resistor_SMD:R_0402_1005Metric, F.Cu at (146.7, 86.0)
- added R12: 1K, Resistor_SMD:R_0402_1005Metric, F.Cu at (146.7, 88.0)
- added R13: 1K, Resistor_SMD:R_0402_1005Metric, F.Cu at (146.7, 90.0)
- added R14: 1K, Resistor_SMD:R_0402_1005Metric, F.Cu at (146.7, 91.9)
- added R2: 5K1, Resistor_SMD:R_0402_1005Metric, F.Cu at (135.6, 102.4)
- added R3: 5K1, Resistor_SMD:R_0402_1005Metric, F.Cu at (139.9, 62.0)
- added R4: 5K1, Resistor_SMD:R_0402_1005Metric, F.Cu at (139.9, 64.0)
- added R5: 2K7, Resistor_SMD:R_0402_1005Metric, F.Cu at (139.9, 66.0)
- added R6: 1K, Resistor_SMD:R_0402_1005Metric, F.Cu at (139.9, 67.9)
- added R7: 1K5, Resistor_SMD:R_0402_1005Metric, F.Cu at (139.9, 69.9)
- added R8: 1K5, Resistor_SMD:R_0402_1005Metric, F.Cu at (139.9, 71.9)
- added R9: 1M, Resistor_SMD:R_0603_1608Metric, F.Cu at (125.1, 75.0)
- added SW1: SW_Push, Button_Switch_SMD:SW_SPST_B3U-3000P, F.Cu at (142.3, 87.8)
- added SW2: SW_Push, Button_Switch_SMD:SW_SPST_B3U-3000P, F.Cu at (142.3, 92.9)
- added SW3: SW_Push, Button_Switch_SMD:SW_SPST_B3U-3000P, F.Cu at (142.3, 98.0)
- added SW4: SW_Push, Button_Switch_SMD:SW_SPST_B3U-3000P, F.Cu at (142.3, 103.0)
- added TP1: ~, TestPoint:TestPoint_Pad_D1.0mm, F.Cu at (132.6, 100.9)
- added TP2: ~, TestPoint:TestPoint_Pad_D1.0mm, F.Cu at (132.6, 104.0)
- added TP3: ~, TestPoint:TestPoint_Pad_D1.0mm, F.Cu at (150.8, 73.0)
- added TP4: ~, TestPoint:TestPoint_Pad_D1.0mm, F.Cu at (150.8, 76.1)
- added U1: W25Q128JVP, Package_SON:WSON-8-1EP_6x5mm_P1.27mm_EP3.4x4.3mm, F.Cu at (129.0, 96.1)
- added U2: STM32WB55CGUx, Package_DFN_QFN:QFN-48-1EP_7x7mm_P0.5mm_EP5.6x5.6mm, F.Cu at (120.1, 89.6)
- added U3: MLPF-WB55-01E3, LibraryFootprints:MLPF-WB55-01E3, F.Cu at (135.7, 104.8)
- added U4: USBLC6-2SC6, Package_TO_SOT_SMD:SOT-23-6, F.Cu at (154.9, 73.9)
- added U5: BQ24090DGQ, LibraryFootprints:MLPF-WB55-01E3, F.Cu at (147.2, 79.5)
- added U6: MAX17048G, Package_DFN_QFN:TDFN-8-1EP_2x2mm_P0.5mm_EP0.8x1.2mm, F.Cu at (143.5, 79.9)
- added U7: TPS7A0508PDBZ, Package_TO_SOT_SMD:SOT-23, F.Cu at (154.8, 78.3)
- added X1: 32MHz, Crystal:Crystal_SMD_2016-4Pin_2.0x1.6mm, F.Cu at (126.8, 104.4)
- added X2: 32kHz768, Crystal:Crystal_SMD_2012-2Pin_2.0x1.2mm, F.Cu at (134.8, 94.5)
Other:
- copper layers 2 -> 4
- rule pad_to_mask_clearance: 0 -> 0.08
