File: 2tonewatch.kicad_pcb (KiCad board)
At the start: 4 copper layers, 58 parts, among them IC1 MDBT50Q-P1MV2, J2 USB_C_Receptacle_USB2.0_16P, J3 Conn_01x02_Pin, J4 FFC-FPC_1X24_PIN, J5 Conn_01x04, Q1 Si1308EDL, SW1 SW_Push, SW2 SW_Push, SW3 SW_Push, SW4 SW_Push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

Commit message: update netlabel colors
Parts:
- removed the J2 at (169.3, 128.4)
- removed the J2 at (147.5, 128.7)
- removed the J2 at (158.2, 128.7)
- removed the J2 at (136.0, 128.7)
- moved C22 18.2 mm to (138.8, 108.8), turned to 0 degrees
- moved C25 15.8 mm to (125.8, 104.5)
- moved L3 13.3 mm to (136.5, 111.2), turned to 180 degrees
- moved C24 12.8 mm to (128.0, 103.8), turned to 0 degrees
- moved J3 12.0 mm to (111.0, 112.2)
- moved J5 12.0 mm to (108.5, 98.4)
- moved D3 5.71 mm to (129.1, 107.0)
- moved R10 3.61 mm to (133.3, 104.6), turned to -90 degrees
- moved Q1 2.00 mm to (135.5, 105.0), turned to -90 degrees
- moved R9 1.21 mm to (137.6, 104.6), turned to -90 degrees

Commit message: Layout progress
Parts:
- removed C16: 1uF, Capacitor_SMD:C_0402_1005Metric
- removed J2: USB_C_Receptacle_USB2.0_16P, Connector_USB:USB_C_Receptacle_Molex_105450-0101
- removed R3, R4: 5K1, Resistor_SMD:R_0402_1005Metric
- removed R5: 2K7, Resistor_SMD:R_0402_1005Metric
- removed R6: 1K, Resistor_SMD:R_0402_1005Metric
- removed R7, R8: 1K5, Resistor_SMD:R_0402_1005Metric
- removed U4: USBLC6-2SC6, Package_TO_SOT_SMD:SOT-23-6
- removed U5: BQ24090DGQ, Package_SO:HVSSOP-10-1EP_3x3mm_P0.5mm_EP1.83x1.89mm
- moved J5 66.6 mm to (174.4, 88.8), turned to 90 degrees
- moved C29 21.2 mm to (123.2, 108.8), turned to 180 degrees
- moved C26 14.5 mm to (123.2, 107.2), turned to 180 degrees
- moved C27 13.2 mm to (123.2, 105.6), turned to 180 degrees
- moved C21 11.2 mm to (133.0, 108.8)
- moved C23 7.49 mm to (123.2, 104.0)
- moved C28 7.14 mm to (119.7, 112.0), turned to -90 degrees
- moved D1 6.12 mm to (125.2, 111.0)
- moved D2 3.03 mm to (125.2, 113.5), turned to 0 degrees
